Commit message: Update lite_6_robotarm.urdf

File: lite_6_robotarm.urdf (robot description, URDF)
Before this commit: robot lite_6_robotarm, 11 links, 10 joints
Links:
- added link baseLink, mass .0; collision box size=1.5 1 0.05; visual mesh filename=table.obj scale=0.1 0.1 0.58

Commit message: Update lite_6_robotarm.urdf

File: lite_6_robotarm.urdf (robot description, URDF)
Before this commit: robot lite_6_robotarm, 12 links, 10 joints
Joints:
- added joint table_robotarm: type continuous, parent baseLink, child base_link, origin xyz=-1.4819862268024002e-06 -0.00020774933500536933 0 rpy=0 0 0, axis -0.0 1.0 -0.0
