Commit message: 주석 추가
각도제한 관련 주석 추가(아랫부분에 있음)

File: lite_6_robotarm-revise.urdf (robot description, URDF)
Before this commit: robot lite_6_robotarm, 11 links, 10 joints
Links:
- removed link camera1
- added link camera_top1, mass 0.2214912391329027; collision mesh filename=meshes/camera_top1.stl scale=0.001 0.001 0.001; visual mesh filename=meshes/camera_top1.stl scale=0.001 0.001 0.001
Joints:
- removed joint base_link_joint
- removed joint left_finger_joint
- removed joint right_finger_joint
- added joint base_link2: type revolute, parent base_link, child link_21, origin xyz=0.0 0.008 0.173 rpy=0 0 0, axis 0.0 -0.0 1.0, limit lower=-6.26 upper=6.26 effort=0.1 velocity=0.1
- added joint left_gripper: type revolute, parent gripper_mount1, child right_finger1, origin xyz=0.026 -0.011 -0.0795 rpy=0 0 0, axis -0.0 1.0 -0.0, limit lower=0.0 upper=1.57 effort=0.1 velocity=0.1
- added joint right_gripper: type revolute, parent gripper_mount1, child left_finger1, origin xyz=-0.026 -0.011 -0.0795 rpy=0 0 0, axis -0.0 1.0 -0.0, limit lower=-1.57 upper=0.0 effort=0.1 velocity=0.1
- joint link2_link3: limit (none) -> lower=-2.09 upper=0.26 effort=0.1 velocity=0.1; type continuous -> revolute
- joint link3_link4: limit (none) -> lower=0.2 upper=2.09 effort=0.1 velocity=0.1; type continuous -> revolute
- joint link4_link5: limit (none) -> lower=-6.26 upper=6.26 effort=0.1 velocity=0.1; type continuous -> revolute
- joint link5_link6: limit (none) -> lower=-1.57 upper=0.78 effort=0.1 velocity=0.1; type continuous -> revolute
- joint link6_link7: limit (none) -> lower=-6.26 upper=6.26 effort=0.1 velocity=0.1; type continuous -> revolute
- joint link7_gripper: type continuous -> fixed
